Commit message: Add camera and lidar town avoidance demo

File: simple_avoidance_sim/urdf/simple_car.urdf.xacro (robot description, xacro)
@@ -274,7 +274,7 @@
   </link>
   <joint name="laser_joint" type="fixed">
-    <parent link="base_link"/>
-    <child link="laser_link"/>
-    <origin xyz="${0.35 * scale} 0 ${0.42 * scale}" rpy="0 0 0"/>
+      <parent link="base_link"/>
+      <child link="laser_link"/>
+      <origin xyz="${0.65 * scale} 0 ${0.38 * scale}" rpy="0 0 0"/>
   </joint>
   <!-- ========================= -->
@@ -309,5 +309,5 @@
     <parent link="base_link"/>
     <child link="camera_link"/>
-    <origin xyz="${0.5 * scale} 0 ${0.42 * scale}" rpy="0 0 0"/>
+    <origin xyz="${0.45 * scale} 0 ${0.52 * scale}" rpy="0 0 0"/>
   </joint>
   <!-- ========================= -->
